Commit message: add self-defined joint state information

File: nusim/urdf/turtlebot3_burger.urdf.xacro (robot description, xacro)
@@ -6,4 +6,5 @@
   <xacro:property name="wheel_radius" value="${props['wheel_radius']}" />
   <xacro:property name="track_width" value="${props['track_width']}"/>
+  <xacro:property name="collision_radius" value="${props['collision_radius']}"/>
   <xacro:arg name ="color" default="black"/>
   <xacro:property name = "color" value = "$(arg color)"/>
@@ -20,10 +21,16 @@
         <mesh filename="package://nuturtle_description/meshes/burger_base.stl" scale="0.001 0.001 0.001"/>
       </geometry>
-      <material name="light_black"/>
+      <material name="${color}"/>
     </visual>
     <collision>
       <origin xyz="-0.032 0 0.070" rpy="0 0 0"/>
       <geometry>
-        <box size="0.140 0.140 0.143"/>
+        <xacro:if value="${collision_radius==0.0}">
+          <box size="0.140 0.140 0.143"/>
+        </xacro:if>
+        <xacro:unless value="${collision_radius ==0.0}">
+          <cylinder radius="${collision_radius}" length="0.23"/>
+        </xacro:unless>
+        <!-- <cylinder radius="0.12" length="0.23"/> -->
       </geometry>
     </collision>
@@ -48,5 +55,5 @@
         <mesh filename="package://nuturtle_description/meshes/left_tire.stl" scale="0.001 0.001 0.001"/>
       </geometry>
-      <material name="${color}"/>
+      <material name="light_black"/>
     </visual>
     <collision>
@@ -76,5 +83,5 @@
         <mesh filename="package://nuturtle_description/meshes/right_tire.stl" scale="0.001 0.001 0.001"/>
       </geometry>
-      <material name="${color}"/>
+      <material name="light_black"/>
     </visual>
     <collision>
@@ -129,5 +136,5 @@
         <mesh filename="package://nuturtle_description/meshes/lds.stl" scale="0.001 0.001 0.001"/>
       </geometry>
-      <material name="${color}"/>
+      <material name="light_black"/>
     </visual>
     <collision>
